Commit message: hexa_tilt

File: models/rotors_description/urdf/hexa_tilt/hexa_tilt.xacro (robot description, xacro)
@@ -2,5 +2,5 @@
 <robot name="iris" xmlns:xacro="http://ros.org/wiki/xacro">
    <!-- Properties -->
-  <xacro:property name="namespace" value="hexa" />
+  <xacro:property name="namespace" value="hexa_tilt" />
   <xacro:property name="rotor_velocity_slowdown_sim" value="10" />
   <xacro:property name="mesh_file" value="hexa.stl" />
@@ -30,4 +30,5 @@
   <xacro:include filename="$(arg rotors_description_dir)/urdf/include/multirotor_base.xacro" />
   <xacro:include filename="$(arg rotors_description_dir)/urdf/include/sensors.xacro" />
+  <xacro:include filename="$(arg rotors_description_dir)/urdf/include/tilt_rotor.xacro" />
   <!-- Property Blocks -->
   <xacro:property name="body_inertia">
@@ -112,5 +113,5 @@
 					</inertial>
 		</link>
-  <xacro:vertical_rotor
+  <xacro:vertical_tilting_rotor
     robot_namespace="${namespace}"
     suffix="3"
@@ -132,6 +133,6 @@
     <origin xyz="0.211396 0.119762 0.082219" rpy="0 0 0" />
     <xacro:insert_block name="rotor_inertia" />
-  </xacro:vertical_rotor>
-   <xacro:vertical_rotor
+  </xacro:vertical_tilting_rotor>
+   <xacro:vertical_tilting_rotor
     robot_namespace="${namespace}"
     suffix="0"
@@ -153,6 +154,6 @@
     <origin xyz="-0.209396 0.122762 0.082219" rpy="0 0 0" />
     <xacro:insert_block name="rotor_inertia" />
-  </xacro:vertical_rotor>
-   <xacro:vertical_rotor
+  </xacro:vertical_tilting_rotor>
+   <xacro:vertical_tilting_rotor
     robot_namespace="${namespace}"
     suffix="4"
@@ -174,6 +175,6 @@
     <origin xyz="-0.00187896 0.242705 0.0822169" rpy="0 0 0" />
     <xacro:insert_block name="rotor_inertia" />
-  </xacro:vertical_rotor>
-  <xacro:vertical_rotor
+  </xacro:vertical_tilting_rotor>
+  <xacro:vertical_tilting_rotor
     robot_namespace="${namespace}"
     suffix="1"
@@ -195,6 +196,6 @@
     <origin xyz="0.211396 -0.119762 0.082219" rpy="0 0 0" />
    <xacro:insert_block name="rotor_inertia" />
-  </xacro:vertical_rotor>
-  <xacro:vertical_rotor
+  </xacro:vertical_tilting_rotor>
+  <xacro:vertical_tilting_rotor
     robot_namespace="${namespace}"
     suffix="5"
@@ -216,6 +217,6 @@
     <origin xyz="-0.00187896 -0.242705 0.0822169" rpy="0 0 0" />
     <xacro:insert_block name="rotor_inertia" />
-  </xacro:vertical_rotor>
-  <xacro:vertical_rotor
+  </xacro:vertical_tilting_rotor>
+  <xacro:vertical_tilting_rotor
     robot_namespace="${namespace}"
     suffix="2"
@@ -237,4 +238,4 @@
     <origin xyz="-0.209396 -0.122762 0.082219" rpy="0 0 0" />
     <xacro:insert_block name="rotor_inertia" />
-  </xacro:vertical_rotor>
+  </xacro:vertical_tilting_rotor>
 </robot>

File: models/rotors_description/urdf/hexa_tilt/hexa_tilt_base.xacro (robot description, xacro)
@@ -1,5 +1,5 @@
 <?xml version="1.0" ?>
 <robot name="hexa" xmlns:xacro="http://ros.org/wiki/xacro">
-	<xacro:arg name='name' default='hexa' />
+	<xacro:arg name='name' default='hexa_tilt' />
 	<xacro:arg name='mavlink_addr' default='INADDR_ANY' />
 	<xacro:arg name='mavlink_udp_port' default='14560' />
@@ -104,3 +104,9 @@
     <origin xyz="0 0 0" rpy="0 0 0" />
   </xacro:imu_plugin_macro>
+	<gazebo>
+		<plugin name="gazebo_ros_control" filename="libgazebo_ros_control.so">
+		  <robotNamespace>tilt</robotNamespace>
+		  <legacyModeNS>true</legacyModeNS>
+		</plugin>
+	</gazebo>
 </robot>

File: models/rotors_description/urdf/include/component_snippets.xacro (robot description, xacro)
@@ -17,5 +17,5 @@
 -->
 <robot xmlns:xacro="http://ros.org/wiki/xacro">
-  <xacro:macro name="ros_interface_macro" params="namespace imu_sub_topic gps_sub_topic">
+  <xacro:macro name="ros_interface_macro" params="namespace imu_sub_topic gps_sub_topic motor_size">
     <gazebo>
       <plugin name="ros_interface" filename="libgazebo_ros_interface.so">
@@ -23,4 +23,5 @@
 				<imuSubTopic>${imu_sub_topic}</imuSubTopic>
         <gpsSubTopic>${gps_sub_topic}</gpsSubTopic>
+        <motorSize>${motor_size}</motorSize>
         <motorSpeedCommandPubTopic>/gazebo/command/motor_speed</motorSpeedCommandPubTopic>
         <control_channels>

File: models/rotors_description/urdf/tarot_tilt/tarot_tilt.xacro (robot description, xacro)
@@ -137,5 +137,6 @@
     <xacro:insert_block name="rotor_inertia" />
   </xacro:vertical_tilting_rotor>
-  <xacro:vertical_tilting_rotor robot_namespace="${namespace}"
+  <xacro:vertical_tilting_rotor
+		robot_namespace="${namespace}"
     suffix="front_left"
     direction="cw"
@@ -157,5 +158,6 @@
     <xacro:insert_block name="rotor_inertia" />
   </xacro:vertical_tilting_rotor>
-  <xacro:vertical_tilting_rotor robot_namespace="${namespace}"
+  <xacro:vertical_tilting_rotor
+		robot_namespace="${namespace}"
     suffix="back_right"
     direction="cw"

File: models/rotors_description/urdf/tarot_tilt/tarot_tilt_base.xacro (robot description, xacro)
@@ -37,5 +37,6 @@
     namespace="${namespace}"
     imu_sub_topic="/imu"
-    gps_sub_topic="/gps">
+    gps_sub_topic="/gps"
+    motor_size="4" >
   </xacro:ros_interface_macro>
   <!-- Instantiate magnetometer plugin. -->
