Commit message: actively tilting firefly added

File: models/rotors_description/urdf/hexa/hexa_base.xacro (robot description, xacro)
@@ -56,4 +56,5 @@
       imu_sub_topic="/imu"
       gps_sub_topic="/gps"
+			odometry_fixed_frame="NED"
       motor_size="6">
     </xacro:ros_interface_macro>

File: models/rotors_description/urdf/hexa_tilt/hexa_tilt_base.xacro (robot description, xacro)
@@ -56,4 +56,5 @@
       imu_sub_topic="/imu"
       gps_sub_topic="/gps"
+			odometry_fixed_frame="NED"
       motor_size="6">
     </xacro:ros_interface_macro>

File: models/rotors_description/urdf/include/component_snippets.xacro (robot description, xacro)
@@ -17,5 +17,5 @@
 -->
 <robot xmlns:xacro="http://ros.org/wiki/xacro">
-  <xacro:macro name="ros_interface_macro" params="namespace imu_sub_topic gps_sub_topic motor_size">
+  <xacro:macro name="ros_interface_macro" params="namespace imu_sub_topic gps_sub_topic odometry_fixed_frame motor_size">
     <gazebo>
       <plugin name="ros_interface" filename="libgazebo_ros_interface.so">
@@ -23,4 +23,5 @@
 				<imuSubTopic>${imu_sub_topic}</imuSubTopic>
         <gpsSubTopic>${gps_sub_topic}</gpsSubTopic>
+				<odomFrame>${odometry_fixed_frame}</odomFrame>
         <motorSize>${motor_size}</motorSize>
         <motorSpeedCommandPubTopic>/gazebo/command/motor_speed</motorSpeedCommandPubTopic>

File: models/rotors_description/urdf/iris_smc/iris_smc_base.xacro (robot description, xacro)
@@ -75,4 +75,5 @@
 		  imu_sub_topic="/imu"
 		  gps_sub_topic="/gps"
+			odometry_fixed_frame="NED"
 		  motor_size="4" >
   	</xacro:ros_interface_macro>

File: models/rotors_description/urdf/tarot_tilt/tarot_tilt_base.xacro (robot description, xacro)
@@ -38,4 +38,5 @@
     imu_sub_topic="/imu"
     gps_sub_topic="/gps"
+		odometry_fixed_frame="NED"
     motor_size="4" >
   </xacro:ros_interface_macro>
