Commit message: with arm uav

File: models/rotors_description/urdf/include/component_snippets.xacro (robot description, xacro)
@@ -674,5 +674,5 @@
         <update_rate>${frame_rate}</update_rate>
         <camera>
-          <horizontal_fov>2</horizontal_fov>
+          <horizontal_fov>1.5</horizontal_fov>
           <image>
             <format>L8</format>
@@ -681,6 +681,6 @@
           </image>
           <clip>
-            <near>0.01</near>
-            <far>100</far>
+            <near>0.2</near>
+            <far>25</far>
           </clip>
         </camera>

File: models/rotors_description/urdf/iris/iris.xacro (robot description, xacro)
@@ -46,4 +46,33 @@
   <!-- Included URDF Files -->
   <xacro:include filename="$(arg rotors_description_dir)/urdf/include/multirotor_base.xacro" />
+  <xacro:include filename="$(arg rotors_description_dir)/urdf/include/sensors.xacro" />
+		<xacro:camera_macro
+				namespace="${namespace}"
+				parent_link="base_link"
+				camera_suffix="raw"
+				frame_rate="30"
+				horizontal_fov="1.4"
+				image_width="1280"
+				image_height="720"
+				image_format="B8G8R8"
+				min_distance="0.02"
+				max_distance="300"
+				noise_mean="0.0"
+				noise_stddev="0.008"
+				enable_visual="1"
+			>
+			<box size="0.02 0.02 0.02" />
+			<origin xyz="0.0 0 -0.04" rpy="0.0 1.57 0.0" />
+		</xacro:camera_macro>
+		<!--
+		<xacro:xtion_pro_live name="rgbd_camera" parent="base_link">
+			<origin xyz="0.11 0.0 -0.02" rpy="0.0 0.95 0.0"/>
+			<origin xyz="0 0 0" rpy="0.0 0 0.0"/>
+		</xacro:xtion_pro_live>
+		-->
+		<xacro:xtion_pro_live name="rgbd_camera" parent="base_link">
+			<origin xyz="0.11 0.0 -0.02" rpy="0.0 0.0 0.0"/>
+			<origin xyz="0 0 0" rpy="0.0 0 0.0"/>
+		</xacro:xtion_pro_live>
   <!-- Instantiate multirotor_base_macro once -->
   <xacro:multirotor_base_macro

File: models/rotors_description/urdf/iris/iris_base.xacro (robot description, xacro)
@@ -68,5 +68,4 @@
     >
   </xacro:barometer_plugin_macro>
-  <xacro:if value="$(arg enable_mavlink_interface)">
   <!-- Instantiate mavlink telemetry interface. -->
   <xacro:mavlink_interface_macro
@@ -95,5 +94,4 @@
     >
   </xacro:mavlink_interface_macro>
-  </xacro:if>
   <!-- Mount an ADIS16448 IMU. -->
   <xacro:imu_plugin_macro
