Commit message: simulatore di ndt2 funzionante

File: models/rotors_description/urdf/include/ndt2_rotor.xacro (robot description, xacro)
@@ -1,4 +1,60 @@
 <?xml version="1.0"?>
 <robot xmlns:xacro="http://ros.org/wiki/xacro">
+  <!-- Main multirotor link -->
+  <xacro:macro name="multirotor_base_macro"
+    params="robot_namespace mass body_width body_height mesh_file mesh_scale color *inertia">
+    <link name="base_link"></link>
+    <joint name="base_joint" type="fixed">
+      <origin xyz="0 0 0" rpy="0 0 0" />
+      <parent link="base_link" />
+      <child link="base_link_inertia" />
+    </joint>
+    <link name="base_link_inertia">
+      <inertial>
+        <mass value="${mass}" />  <!-- [kg] -->
+        <origin xyz="0 0 0" />
+        <xacro:insert_block name="inertia" />
+      </inertial>
+      <visual>
+        <origin xyz="0 0 0" rpy="0 0 0" />
+        <geometry>
+          <mesh filename="package://rotors_description/meshes/${mesh_file}"
+            scale="${mesh_scale}" />
+          <!-- <box size="${body_width} ${body_width} ${body_height}"/> --> <!-- [m] [m] [m] -->
+        </geometry>
+      </visual>
+      <collision>
+        <origin xyz="0 0 0" rpy="0 0 0" />
+        <geometry>
+          <mesh filename="package://rotors_description/meshes/${mesh_file}"
+            scale="${mesh_scale}" />
+        </geometry>
+      </collision>
+    </link>
+    <!-- attach multirotor_base_plugin to the base_link -->
+    <gazebo>
+      <plugin filename="libgazebo_multirotor_base_plugin.so" name="rosbag">
+        <robotNamespace>${robot_namespace}</robotNamespace>
+        <linkName>base_link</linkName>
+        <rotorVelocitySlowdownSim>${rotor_velocity_slowdown_sim}</rotorVelocitySlowdownSim>
+      </plugin>
+    </gazebo>
+    <gazebo reference="base_link">
+      <material>Gazebo/${color}</material>
+      <collision name='base_link_inertia_collision'>
+        <surface>
+          <contact>
+            <ode>
+              <min_depth>0.001</min_depth>
+              <max_vel>0.0</max_vel>
+            </ode>
+          </contact>
+          <friction>
+            <ode/>
+          </friction>
+        </surface>
+      </collision>
+   </gazebo>
+  </xacro:macro>
 <!-- Rotor joint and link -->
   <xacro:macro name="vertical_rotor"

File: models/rotors_description/urdf/ndt2/ndt2.xacro (robot description, xacro)
@@ -1,5 +1,5 @@
 <?xml version="1.0" ?>
 <robot name="ndt2" xmlns:xacro="http://www.ros.org/wiki/xacro">
-  <xacro:property name="namespace" value="" />
+  <xacro:property name="namespace" value="ndt2" />
   <xacro:property name="mass" value="6.0" /> <!-- [kg] -->
   <xacro:property name="body_width" value="1.0" /> <!-- [m] -->
@@ -26,9 +26,9 @@
   <xacro:property name="x_rotor" value="0.121"  />
   <xacro:property name="y_rotor" value="0.121"  />
-  <xacro:property name="z_rotor" value="0.068"  />
+  <xacro:property name="z_rotor" value="0.075"  />
   <xacro:include filename="$(arg rotors_description_dir)/urdf/ndt2/ndt2.trans" />
   <xacro:include filename="$(arg rotors_description_dir)/urdf/ndt2/ndt2.gazebo" />
-	<xacro:include filename="$(arg rotors_description_dir)/urdf/include/multirotor_base.xacro" />
   <xacro:include filename="$(arg rotors_description_dir)/urdf/include/ndt2_rotor.xacro" />
+  <!--<xacro:include filename="$(arg rotors_description_dir)/urdf/include/multirotor_base.xacro" />-->
   <xacro:include filename="$(arg rotors_description_dir)/urdf/include/sensors.xacro" />
   <xacro:property name="body_inertia">
@@ -175,5 +175,5 @@
   <xacro:vertical_rotor
     robot_namespace="${namespace}"
-    suffix="1"
+    suffix="0"
     direction="cw"
     motor_constant="${motor_constant}"
@@ -185,5 +185,5 @@
     time_constant_down="${time_constant_down}"
     max_rot_velocity="${max_rot_velocity}"
-    motor_number="1"
+    motor_number="0"
     rotor_drag_coefficient="${rotor_drag_coefficient}"
     rolling_moment_coefficient="${rolling_moment_coefficient}"
@@ -196,5 +196,5 @@
   <xacro:vertical_rotor
     robot_namespace="${namespace}"
-    suffix="2"
+    suffix="1"
     direction="ccw"
     motor_constant="${motor_constant}"
@@ -206,5 +206,5 @@
     time_constant_down="${time_constant_down}"
     max_rot_velocity="${max_rot_velocity}"
-    motor_number="2"
+    motor_number="1"
     rotor_drag_coefficient="${rotor_drag_coefficient}"
     rolling_moment_coefficient="${rolling_moment_coefficient}"
@@ -217,5 +217,5 @@
   <xacro:vertical_rotor
     robot_namespace="${namespace}"
-    suffix="3"
+    suffix="2"
     direction="cw"
     motor_constant="${motor_constant}"
@@ -227,5 +227,5 @@
     time_constant_down="${time_constant_down}"
     max_rot_velocity="${max_rot_velocity}"
-    motor_number="3"
+    motor_number="2"
     rotor_drag_coefficient="${rotor_drag_coefficient}"
     rolling_moment_coefficient="${rolling_moment_coefficient}"
@@ -238,9 +238,31 @@
   <xacro:vertical_rotor
     robot_namespace="${namespace}"
+    suffix="3"
+    direction="ccw"
+    motor_constant="${motor_constant}"
+    moment_constant="${moment_constant}"
+    parent="arm_4"
+    mass_rotor="${mass_rotor}"
+    radius_rotor="${radius_rotor}"
+    time_constant_up="${time_constant_up}"
+    time_constant_down="${time_constant_down}"
+    max_rot_velocity="${max_rot_velocity}"
+    motor_number="3"
+    rotor_drag_coefficient="${rotor_drag_coefficient}"
+    rolling_moment_coefficient="${rolling_moment_coefficient}"
+    mesh="prop.stl"
+    mesh_scale="${mesh_scale}"
+    color="Blue">
+    <origin xyz="${x_rotor} -${y_rotor} ${z_rotor}" rpy="0 0 0" />
+    <xacro:insert_block name="rotor_inertia" />
+  </xacro:vertical_rotor>
+  <!-- Bottom layer of rotors-->
+  <xacro:vertical_rotor
+    robot_namespace="${namespace}"
     suffix="4"
     direction="ccw"
     motor_constant="${motor_constant}"
     moment_constant="${moment_constant}"
-    parent="arm_4"
+    parent="arm_1"
     mass_rotor="${mass_rotor}"
     radius_rotor="${radius_rotor}"
@@ -249,26 +271,4 @@
     max_rot_velocity="${max_rot_velocity}"
     motor_number="4"
-    rotor_drag_coefficient="${rotor_drag_coefficient}"
-    rolling_moment_coefficient="${rolling_moment_coefficient}"
-    mesh="prop.stl"
-    mesh_scale="${mesh_scale}"
-    color="Blue">
-    <origin xyz="${x_rotor} -${y_rotor} ${z_rotor}" rpy="0 0 0" />
-    <xacro:insert_block name="rotor_inertia" />
-  </xacro:vertical_rotor>
-  <!-- Bottom layer of rotors-->
-  <xacro:vertical_rotor
-    robot_namespace="${namespace}"
-    suffix="5"
-    direction="ccw"
-    motor_constant="${motor_constant}"
-    moment_constant="${moment_constant}"
-    parent="arm_1"
-    mass_rotor="${mass_rotor}"
-    radius_rotor="${radius_rotor}"
-    time_constant_up="${time_constant_up}"
-    time_constant_down="${time_constant_down}"
-    max_rot_velocity="${max_rot_velocity}"
-    motor_number="5"
     rotor_drag_coefficient="${rotor_drag_coefficient}"
     rolling_moment_coefficient="${rolling_moment_coefficient}"
@@ -281,5 +281,5 @@
   <xacro:vertical_rotor
     robot_namespace="${namespace}"
-    suffix="6"
+    suffix="5"
     direction="cw"
     motor_constant="${motor_constant}"
@@ -291,5 +291,5 @@
     time_constant_down="${time_constant_down}"
     max_rot_velocity="${max_rot_velocity}"
-    motor_number="6"
+    motor_number="5"
     rotor_drag_coefficient="${rotor_drag_coefficient}"
     rolling_moment_coefficient="${rolling_moment_coefficient}"
@@ -302,5 +302,5 @@
   <xacro:vertical_rotor
     robot_namespace="${namespace}"
-    suffix="7"
+    suffix="6"
     direction="ccw"
     motor_constant="${motor_constant}"
@@ -312,5 +312,5 @@
     time_constant_down="${time_constant_down}"
     max_rot_velocity="${max_rot_velocity}"
-    motor_number="7"
+    motor_number="6"
     rotor_drag_coefficient="${rotor_drag_coefficient}"
     rolling_moment_coefficient="${rolling_moment_coefficient}"
@@ -323,5 +323,5 @@
   <xacro:vertical_rotor
     robot_namespace="${namespace}"
-    suffix="8"
+    suffix="7"
     direction="cw"
     motor_constant="${motor_constant}"
@@ -333,5 +333,5 @@
     time_constant_down="${time_constant_down}"
     max_rot_velocity="${max_rot_velocity}"
-    motor_number="8"
+    motor_number="7"
     rotor_drag_coefficient="${rotor_drag_coefficient}"
     rolling_moment_coefficient="${rolling_moment_coefficient}"

File: models/rotors_description/urdf/ndt2/ndt2_base.xacro (robot description, xacro)
@@ -23,5 +23,5 @@
   <xacro:arg name='vehicle_is_tailsitter' default='false' />
   <xacro:arg name='visual_material' default='DarkGrey' />
-  <xacro:arg name='enable_mavlink_interface' default='true' />
+  <xacro:arg name='enable_mavlink_interface' default='false' />
   <xacro:arg name='enable_wind' default='false' />
   <!-- The following causes segfault with multiple vehicles if defaults to true!!! -->
@@ -68,4 +68,12 @@
     >
   </xacro:barometer_plugin_macro>
+  <xacro:ros_interface_macro
+		  namespace="${namespace}"
+		  imu_sub_topic="/imu"
+		  gps_sub_topic="/gps"
+			odometry_fixed_frame="NED"
+		  motor_size="8" >
+  	</xacro:ros_interface_macro>
+  <xacro:if value="$(arg enable_mavlink_interface)">
   <!-- Instantiate mavlink telemetry interface. -->
   <xacro:mavlink_interface_macro
@@ -94,4 +102,5 @@
     >
   </xacro:mavlink_interface_macro>
+  </xacro:if>
   <!-- Mount an ADIS16448 IMU. -->
   <xacro:imu_plugin_macro
@@ -173,3 +182,9 @@
     </xacro:bag_plugin_macro>
   </xacro:if>
+ <gazebo>
+    <plugin name="gazebo_ros_control" filename="libgazebo_ros_control.so">
+      <robotNamespace>ndt2</robotNamespace>
+      <legacyModeNS>true</legacyModeNS>
+    </plugin>
+  </gazebo>
 </robot>
