Commit message: ndt2 final commit

File: models/rotors_description/urdf/include/_d435.urdf.xacro (robot description, xacro)
@@ -7,3 +7,115 @@
 -->
 <robot name="sensor_d435" xmlns:xacro="http://ros.org/wiki/xacro">
+  <!--File includes-->
+  <xacro:include filename="$(arg rotors_description_dir)/urdf/include/_d435.gazebo.xacro"/>
+	<xacro:property name="M_PI" value="3.1415926535897931" />
+    <!-- The following values are approximate, and the camera node
+     publishing TF values with actual calibrated camera extrinsic values -->
+    <xacro:property name="d435_cam_depth_to_left_ir_offset" value="0.0"/>
+    <xacro:property name="d435_cam_depth_to_right_ir_offset" value="-0.050"/>
+    <xacro:property name="d435_cam_depth_to_color_offset" value="0.015"/>
+    <!-- The following values model the aluminum peripherial case for the
+  	D435 camera, with the camera joint represented by the actual
+  	peripherial camera tripod mount -->
+    <xacro:property name="d435_cam_width" value="0.090"/>
+    <xacro:property name="d435_cam_height" value="0.025"/>
+    <xacro:property name="d435_cam_depth" value="0.02505"/>
+    <xacro:property name="d435_cam_mount_from_center_offset" value="0.0149"/>
+    <!-- The following offset is relative the the physical D435 camera peripherial
+  	camera tripod mount -->
+    <xacro:property name="d435_cam_depth_px" value="${d435_cam_mount_from_center_offset}"/>
+    <xacro:property name="d435_cam_depth_py" value="0.0175"/>
+    <xacro:property name="d435_cam_depth_pz" value="${d435_cam_height/2}"/>
+  <xacro:macro name="sensor_d435" params="name:=camera topics_ns:=camera parent *origin">
+    <material name="${name}_aluminum">
+	  <color rgba="0.5 0.5 0.5 1"/>
+    </material>
+    <!-- camera body, with origin at bottom screw mount -->
+    <joint name="${name}_joint" type="fixed">
+      <xacro:insert_block name="origin" />
+      <parent link="${parent}"/>
+      <child link="${name}_bottom_screw_frame" />
+    </joint>
+    <link name="${name}_bottom_screw_frame"/>
+    <joint name="${name}_link_joint" type="fixed">
+      <origin xyz="0 ${d435_cam_depth_py} ${d435_cam_depth_pz}" rpy="0 0 0"/>
+      <parent link="${name}_bottom_screw_frame"/>
+      <child link="${name}_link" />
+    </joint>
+    <link name="${name}_link">
+      <visual>
+      <origin xyz="${d435_cam_mount_from_center_offset} ${-d435_cam_depth_py} 0" rpy="${M_PI/2} 0 ${M_PI/2}"/>
+        <geometry>
+          <mesh filename="package://rotors_description/meshes/d435.dae" />
+        </geometry>
+        <material name="${name}_aluminum"/>
+      </visual>
+      <collision>
+        <origin xyz="0 ${-d435_cam_depth_py} 0" rpy="0 0 0"/>
+        <geometry>
+        <box size="${d435_cam_depth} ${d435_cam_width} ${d435_cam_height}"/>
+        </geometry>
+      </collision>
+      <inertial>
+        <!-- The following are not reliable values, and should not be used for modeling -->
+        <mass value="0.0001" />
+        <origin xyz="0 0 0" />
+        <inertia ixx="0.00001" ixy="0.0" ixz="0.0" iyy="0.00001" iyz="0.0" izz="0.00001" />
+      </inertial>
+    </link>
+    <!-- camera depth joints and links -->
+    <joint name="${name}_depth_joint" type="fixed">
+      <origin xyz="0 0 0" rpy="0 0 0"/>
+      <parent link="${name}_link"/>
+      <child link="${name}_depth_frame" />
+    </joint>
+    <link name="${name}_depth_frame"/>
+    <joint name="${name}_depth_optical_joint" type="fixed">
+      <origin xyz="0 0 0" rpy="${-M_PI/2} 0 ${-M_PI/2}" />
+      <parent link="${name}_depth_frame" />
+      <child link="${name}_depth_optical_frame" />
+    </joint>
+    <link name="${name}_depth_optical_frame"/>
+    <!-- camera left IR joints and links -->
+    <joint name="${name}_left_ir_joint" type="fixed">
+      <origin xyz="0 ${d435_cam_depth_to_left_ir_offset} 0" rpy="0 0 0" />
+      <parent link="${name}_depth_frame" />
+      <child link="${name}_left_ir_frame" />
+    </joint>
+    <link name="${name}_left_ir_frame"/>
+    <joint name="${name}_left_ir_optical_joint" type="fixed">
+      <origin xyz="0 0 0" rpy="${-M_PI/2} 0 ${-M_PI/2}" />
+      <parent link="${name}_left_ir_frame" />
+      <child link="${name}_left_ir_optical_frame" />
+    </joint>
+    <link name="${name}_left_ir_optical_frame"/>
+    <!-- camera right IR joints and links -->
+    <joint name="${name}_right_ir_joint" type="fixed">
+      <origin xyz="0 ${d435_cam_depth_to_right_ir_offset} 0" rpy="0 0 0" />
+      <parent link="${name}_depth_frame" />
+      <child link="${name}_right_ir_frame" />
+    </joint>
+    <link name="${name}_right_ir_frame"/>
+    <joint name="${name}_right_ir_optical_joint" type="fixed">
+      <origin xyz="0 0 0" rpy="${-M_PI/2} 0 ${-M_PI/2}" />
+      <parent link="${name}_right_ir_frame" />
+      <child link="${name}_right_ir_optical_frame" />
+    </joint>
+    <link name="${name}_right_ir_optical_frame"/>
+    <!-- camera color joints and links -->
+    <joint name="${name}_color_joint" type="fixed">
+      <origin xyz="0 ${d435_cam_depth_to_color_offset} 0" rpy="0 0 0" />
+      <parent link="${name}_depth_frame" />
+      <child link="${name}_color_frame" />
+    </joint>
+    <link name="${name}_color_frame"/>
+    <joint name="${name}_color_optical_joint" type="fixed">
+      <origin xyz="0 0 0" rpy="${-M_PI/2} 0 ${-M_PI/2}" />
+      <parent link="${name}_color_frame" />
+      <child link="${name}_color_optical_frame" />
+    </joint>
+    <link name="${name}_color_optical_frame"/>
+    <!-- Realsense Gazebo Plugin -->
+    <xacro:gazebo_d435 camera_name="${name}" reference_link="${name}_link" topics_ns="${topics_ns}" depth_optical_frame="${name}_depth_optical_frame" color_optical_frame="${name}_color_optical_frame" infrared1_optical_frame="${name}_left_ir_optical_frame" infrared2_optical_frame="${name}_right_ir_optical_frame"/>
+  </xacro:macro>
 </robot>

File: models/rotors_description/urdf/iris/iris.xacro (robot description, xacro)
@@ -1,4 +1,5 @@
 <?xml version="1.0"?>
 <robot name="iris" xmlns:xacro="http://ros.org/wiki/xacro">
+  <xacro:arg name='rotors_description_dir' default='$(find mavlink_sitl_gazebo)/models/rotors_description' />
   <!-- Properties -->
   <xacro:property name="namespace" value="" />
@@ -27,5 +28,5 @@
   <xacro:property name="rotor_drag_coefficient" value="1.75e-04" />
   <xacro:property name="rolling_moment_coefficient" value="0.000001" />
-  <xacro:property name="color" value="$(arg visual_material)" />
+  <xacro:property name="color" value="white" />
   <!-- Property Blocks -->
   <xacro:property name="body_inertia">
@@ -47,4 +48,6 @@
   <xacro:include filename="$(arg rotors_description_dir)/urdf/include/multirotor_base.xacro" />
   <xacro:include filename="$(arg rotors_description_dir)/urdf/include/sensors.xacro" />
+  <xacro:include filename="$(arg rotors_description_dir)/urdf/include/_d435.urdf.xacro" />
+		<!--
 		<xacro:camera_macro
 				namespace="${namespace}"
@@ -65,14 +68,14 @@
 			<origin xyz="0.0 0 -0.04" rpy="0.0 1.57 0.0" />
 		</xacro:camera_macro>
+		-->
+		<xacro:sensor_d435 parent="base_link" >
+      		<origin xyz="0 0.0 -0.04" rpy="0 1.57 0"/>
+  		</xacro:sensor_d435>
 		<!--
-		<xacro:xtion_pro_live name="rgbd_camera" parent="base_link">
-			<origin xyz="0.11 0.0 -0.02" rpy="0.0 0.95 0.0"/>
-			<origin xyz="0 0 0" rpy="0.0 0 0.0"/>
-		</xacro:xtion_pro_live>
-		-->
 		<xacro:xtion_pro_live name="rgbd_camera" parent="base_link">
 			<origin xyz="0.11 0.0 -0.02" rpy="0.0 0.5 0.0"/>
 			<origin xyz="0 0 0" rpy="0.0 0 0.0"/>
 		</xacro:xtion_pro_live>
+		-->
   <!-- Instantiate multirotor_base_macro once -->
   <xacro:multirotor_base_macro

File: models/rotors_description/urdf/iris/iris_base.xacro (robot description, xacro)
@@ -5,4 +5,5 @@
   -->
   <xacro:arg name='name' default='iris' />
+  <xacro:arg name='rotors_description_dir' default='$(find mavlink_sitl_gazebo)/models/rotors_description' />
   <xacro:arg name='mavlink_addr' default='INADDR_ANY' />
   <xacro:arg name='mavlink_udp_port' default='14560' />

File: models/rotors_description/urdf/ndt2/ndt2.xacro (robot description, xacro)
@@ -15,12 +15,12 @@
   <xacro:property name="radius_rotor" value="0.2545" /> <!-- [m] -->
   <xacro:property name="motor_constant" value="0.00019065" /> <!-- [kg.m/s^2] -->
-  <xacro:property name="moment_constant" value="0.06" /> <!-- [m] -->
+  <xacro:property name="moment_constant" value="0.000001333" /> <!-- 0.06 [m] -->
   <xacro:property name="time_constant_up" value="0.0125" /> <!-- [s] -->
   <xacro:property name="time_constant_down" value="0.025" /> <!-- [s] -->
-  <xacro:property name="max_rot_velocity" value="1100" /> <!-- [rad/s] -->
+  <xacro:property name="max_rot_velocity" value="5000" /> <!-- [rad/s] -->
   <xacro:property name="sin30" value="0.5" />
   <xacro:property name="cos30" value="0.866025403784" />
   <xacro:property name="sqrt2" value="1.4142135623730951" />
-  <xacro:property name="rotor_drag_coefficient" value="0.000001333" />
+  <xacro:property name="rotor_drag_coefficient" value="1.75e-04" />
   <xacro:property name="rolling_moment_coefficient" value="0.000001" />
   <xacro:property name="x_rotor" value="0.121"  />
@@ -144,5 +144,5 @@
     </collision>
   </link>
-  <joint name="tilt_motor_4" type="continuous">
+  <joint name="tilt_motor_4" type="revolute">
     <origin rpy="0 0 0" xyz="0.224433 -0.234052 0.04"/>
     <parent link="base_link"/>
@@ -151,12 +151,12 @@
     <limit effort="30" velocity="1.0" lower="-1.57" upper="1.57"/>
   </joint>
-  <joint name="tilt_motor_2" type="continuous">
+  <joint name="tilt_motor_2" type="revolute">
     <origin rpy="0 0 0" xyz="-0.224433 0.234052 0.04"/>
     <parent link="base_link"/>
     <child link="arm_2"/>
-    <axis xyz="-0.707107 0.707107 -0.0"/>
+    <axis xyz="-0.707107 0.707107 0.0"/>
     <limit effort="30" velocity="1.0" lower="-1.57" upper="1.57"/>
   </joint>
-  <joint name="tilt_motor_3" type="continuous">
+  <joint name="tilt_motor_3" type="revolute">
     <origin rpy="0 0 0" xyz="-0.224433 -0.234052 0.04"/>
     <parent link="base_link"/>
@@ -165,5 +165,5 @@
     <limit effort="30" velocity="1.0" lower="-1.57" upper="1.57"/>
   </joint>
-  <joint name="tilt_motor_1" type="continuous">
+  <joint name="tilt_motor_1" type="revolute">
     <origin rpy="0 0 0" xyz="0.224433 0.234052 0.04"/>
     <parent link="base_link"/>
@@ -190,5 +190,5 @@
     mesh="prop.stl"
     mesh_scale="${mesh_scale}"
-    color="White">
+    color="Blue">
     <origin xyz="${x_rotor} ${y_rotor} ${z_rotor}" rpy="0 0 0" />
     <xacro:insert_block name="rotor_inertia" />
@@ -211,5 +211,5 @@
     mesh="prop.stl"
     mesh_scale="${mesh_scale}"
-    color="Blue">
+    color="White">
     <origin xyz="-${x_rotor} ${y_rotor} ${z_rotor}" rpy="0 0 0" />
     <xacro:insert_block name="rotor_inertia" />
@@ -317,5 +317,5 @@
     mesh="prop.stl"
     mesh_scale="${mesh_scale}"
-    color="Blue">
+    color="White">
     <origin xyz="-${x_rotor} -${y_rotor} -${z_rotor}" rpy="0 0 0" />
     <xacro:insert_block name="rotor_inertia" />
@@ -338,5 +338,5 @@
     mesh="prop.stl"
     mesh_scale="${mesh_scale}"
-    color="White">
+    color="Blue">
     <origin xyz="${x_rotor} -${y_rotor} -${z_rotor}" rpy="0 0 0" />
     <xacro:insert_block name="rotor_inertia" />

File: models/rotors_description/urdf/ndt2/ndt2_base.xacro (robot description, xacro)
@@ -23,5 +23,5 @@
   <xacro:arg name='vehicle_is_tailsitter' default='false' />
   <xacro:arg name='visual_material' default='DarkGrey' />
-  <xacro:arg name='enable_mavlink_interface' default='false' />
+  <xacro:arg name='enable_mavlink_interface' default='true' />
   <xacro:arg name='enable_wind' default='false' />
   <!-- The following causes segfault with multiple vehicles if defaults to true!!! -->

File: models/rotors_description/urdf/tarot/tarot.xacro (robot description, xacro)
@@ -28,9 +28,10 @@
   <xacro:property name="rolling_moment_coefficient" value="0.000001" />
   <xacro:property name="color" value="$(arg visual_material)" />
-	<xacro:arg name='enable_camera' default='false'/>
+  <xacro:arg name='enable_camera' default='true'/>
   <xacro:arg name='enable_depth' default='false' />
   <xacro:arg name='enable_laser' default='false' />
   <xacro:include filename="$(arg rotors_description_dir)/urdf/include/multirotor_base.xacro" />
   <xacro:include filename="$(arg rotors_description_dir)/urdf/include/sensors.xacro" />
+  <xacro:include filename="$(arg rotors_description_dir)/urdf/include/_d435.urdf.xacro" />
   <!-- Property Blocks -->
   <xacro:property name="body_inertia">
@@ -50,5 +51,5 @@
   </xacro:property>
   <xacro:if value="$(arg enable_camera)">
-		<xacro:camera_macro
+		<!--<xacro:camera_macro
 				namespace="${namespace}"
 				parent_link="base_link"
@@ -68,8 +69,12 @@
 			<origin xyz="0.0 0 -0.04" rpy="0.0 1.57 0.0" />
 		</xacro:camera_macro>
+		-->
   </xacro:if>
+  <xacro:sensor_d435 parent="base_link" >
+    <origin xyz="-0.01 0.0 -0.045" rpy="0 1.57 0"/>
+  </xacro:sensor_d435>
   <xacro:if value="$(arg enable_depth)">
 		<xacro:xtion_pro_live name="rgbd_camera" parent="base_link">
-			<origin xyz="0.11 0.0 -0.02" rpy="0.0 0.95 0.0"/>
+			<origin xyz="0.11 0.0 -0.02" rpy="0.0 1.95 0.0"/>
 			<origin xyz="0 0 0" rpy="0.0 0 0.0"/>
 		</xacro:xtion_pro_live>
