Commit message: testing tarot960

File: models/rotors_description/urdf/tarot960/tarot960.xacro (robot description, xacro)
@@ -7,5 +7,5 @@
   <xacro:property name="mesh_scale" value="0.001 0.001 0.001"/>
   <xacro:property name="mesh_scale_prop" value="1 1 1"/>
-  <xacro:property name="mass" value="1.5" /> <!-- [kg] -->
+  <xacro:property name="mass" value="0.5" /> <!-- [kg] -->
   <xacro:property name="body_width" value="0.47" /> <!-- [m] -->
   <xacro:property name="body_height" value="0.11" /> <!-- [m] -->
@@ -17,5 +17,5 @@
   <xacro:property name="rotor_offset_top" value="0.023" /> <!-- [m] -->
   <xacro:property name="radius_rotor" value="0.128" /> <!-- [m] -->
-  <xacro:property name="motor_constant" value="8.54858e-05" /> <!-- [kg.m/s^2] -->
+  <xacro:property name="motor_constant" value="0.00000854858" /> <!-- [kg.m/s^2] -->
   <xacro:property name="moment_constant" value="0.06" /> <!-- [m] -->
   <xacro:property name="time_constant_up" value="0.0125" /> <!-- [s] -->

File: models/rotors_description/urdf/tarot960/tarot960_base.xacro (robot description, xacro)
@@ -86,5 +86,5 @@
   <xacro:if value="$(arg enable_mavlink_interface)">
 -->
-  <!-- Instantiate mavlink telemetry interface. -->
+  <!-- Instantiate mavlink telemetry interface.
   <xacro:mavlink_interface_macro
     namespace="${namespace}"
@@ -112,5 +112,4 @@
     >
   </xacro:mavlink_interface_macro>
-  <!--
 </xacro:if>
 -->
