Commit message: new rotation for depth sensor

File: models/rotors_description/urdf/iris/iris.xacro (robot description, xacro)
@@ -72,5 +72,5 @@
 		-->
 		<xacro:xtion_pro_live name="rgbd_camera" parent="base_link">
-			<origin xyz="0.11 0.0 -0.02" rpy="0.0 0.0 0.0"/>
+			<origin xyz="0.11 0.0 -0.02" rpy="0.0 0.5 0.0"/>
 			<origin xyz="0 0 0" rpy="0.0 0 0.0"/>
 		</xacro:xtion_pro_live>
